Commit message: Added functional IK code, Updated Name of URDF

File: CAD Files+URDFS/URDF/Arm2.urdf (robot description, URDF)
Before this commit: robot WheelChairArm1, 9 links, 8 joints
Joints:
- joint Stepper1Joint: type revolute -> continuous
- joint Stepper2Joint: type revolute -> continuous
- joint Stepper3Joint: type revolute -> continuous
- joint Stepper4Joint: type revolute -> continuous
