Commit message: Adding 7DOF URDF+IK

File: URDF-Model+IK/7DOFArm.SLDASM/urdf/7DOFArm.SLDASM.urdf (robot description, URDF)
Before this commit: robot 5DOFArm, 8 links, 7 joints
Links:
- removed link ConnectingJointA
- removed link ConnectingJointB
- removed link Grapper
- removed link Motor1
- removed link Motor2
- removed link Motor3
- removed link Motor4
- removed link Motor5
- added link EndEffector, mass 0.533035537217521; collision mesh filename=package://7DOFArm.SLDASM/meshes/EndEffector.STL; visual mesh filename=package://7DOFArm.SLDASM/meshes/EndEffector.STL
- added link Link2, mass 0.055389475138638; collision mesh filename=package://7DOFArm.SLDASM/meshes/Link2.STL; visual mesh filename=package://7DOFArm.SLDASM/meshes/Link2.STL
- added link Link3, mass 0.390826093219989; collision mesh filename=package://7DOFArm.SLDASM/meshes/Link3.STL; visual mesh filename=package://7DOFArm.SLDASM/meshes/Link3.STL
- added link Link4, mass 0.055389475138638; collision mesh filename=package://7DOFArm.SLDASM/meshes/Link4.STL; visual mesh filename=package://7DOFArm.SLDASM/meshes/Link4.STL
- added link Link5, mass 0.391896328746283; collision mesh filename=package://7DOFArm.SLDASM/meshes/Link5.STL; visual mesh filename=package://7DOFArm.SLDASM/meshes/Link5.STL
- added link Link6, mass 0.0553894751386379; collision mesh filename=package://7DOFArm.SLDASM/meshes/Link6.STL; visual mesh filename=package://7DOFArm.SLDASM/meshes/Link6.STL
- added link Link7, mass 0.391361210934714; collision mesh filename=package://7DOFArm.SLDASM/meshes/Link7.STL; visual mesh filename=package://7DOFArm.SLDASM/meshes/Link7.STL
- added link base_link, mass 0.195948164313462; collision mesh filename=package://7DOFArm.SLDASM/meshes/base_link.STL; visual mesh filename=package://7DOFArm.SLDASM/meshes/base_link.STL
Joints:
- removed joint ConnectingJoint1
- removed joint ConnectingJointA2
- removed joint ConnectingJointB1
- removed joint ConnectingJointB2
- removed joint Motor2to3Fixed
- removed joint Motor4to5
- removed joint Motor5toGrapper
- added joint Joint0: type continuous, parent base_link, child Link2, origin xyz=0 0.0395 0.044 rpy=0 0 -0.0063255066818594, axis 0 0 1
- added joint Joint1: type continuous, parent Link2, child Link3, origin xyz=0 -0.0030000000000001 0.0450000000000002 rpy=1.06447174148775 0 0, axis 1 0 0
- added joint Joint2: type continuous, parent Link3, child Link4, origin xyz=0 0 0.204 rpy=-0.982875993996659 0 0, axis -1 0 0
- added joint Joint3: type continuous, parent Link4, child Link5, origin xyz=0 0.00300000000000002 0.0339337982667513 rpy=0 0 -0.0373408822518601, axis 0 0 -1
- added joint Joint4: type continuous, parent Link5, child Link6, origin xyz=0 0.140049941199938 0.0340662017332484 rpy=0 0.0178678459046033 0, axis 0 1 0
- added joint Joint5: type continuous, parent Link6, child Link7, origin xyz=0 0.0509500588000616 0.00300000000000006 rpy=-0.00877434456653207 0 0, axis -1 0 0
- added joint Joint6: type continuous, parent Link7, child EndEffector, origin xyz=0.000999999999997949 0.124829928909805 0 rpy=0 0 0, axis 0 -1 0

File: URDF-Model+IK/7DOFArm.urdf (robot description, URDF)
Before this commit: robot 5DOFArm, 8 links, 7 joints
Links:
- removed link ConnectingJointA
- removed link ConnectingJointB
- removed link Grapper
- removed link Motor1
- removed link Motor2
- removed link Motor3
- removed link Motor4
- removed link Motor5
- added link EndEffector, mass 0.533035537217521; collision mesh filename=package://7DOFArm.SLDASM/meshes/EndEffector.STL; visual mesh filename=package://7DOFArm.SLDASM/meshes/EndEffector.STL
- added link Link2, mass 0.055389475138638; collision mesh filename=package://7DOFArm.SLDASM/meshes/Link2.STL; visual mesh filename=package://7DOFArm.SLDASM/meshes/Link2.STL
- added link Link3, mass 0.390826093219989; collision mesh filename=package://7DOFArm.SLDASM/meshes/Link3.STL; visual mesh filename=package://7DOFArm.SLDASM/meshes/Link3.STL
- added link Link4, mass 0.055389475138638; collision mesh filename=package://7DOFArm.SLDASM/meshes/Link4.STL; visual mesh filename=package://7DOFArm.SLDASM/meshes/Link4.STL
- added link Link5, mass 0.391896328746283; collision mesh filename=package://7DOFArm.SLDASM/meshes/Link5.STL; visual mesh filename=package://7DOFArm.SLDASM/meshes/Link5.STL
- added link Link6, mass 0.0553894751386379; collision mesh filename=package://7DOFArm.SLDASM/meshes/Link6.STL; visual mesh filename=package://7DOFArm.SLDASM/meshes/Link6.STL
- added link Link7, mass 0.391361210934714; collision mesh filename=package://7DOFArm.SLDASM/meshes/Link7.STL; visual mesh filename=package://7DOFArm.SLDASM/meshes/Link7.STL
- added link base_link, mass 0.195948164313462; collision mesh filename=package://7DOFArm.SLDASM/meshes/base_link.STL; visual mesh filename=package://7DOFArm.SLDASM/meshes/base_link.STL
Joints:
- removed joint ConnectingJoint1
- removed joint ConnectingJointA2
- removed joint ConnectingJointB1
- removed joint ConnectingJointB2
- removed joint Motor2to3Fixed
- removed joint Motor4to5
- removed joint Motor5toGrapper
- added joint Joint0: type continuous, parent base_link, child Link2, origin xyz=0 0.0395 0.044 rpy=0 0 -0.0063255066818594, axis 0 0 1
- added joint Joint1: type continuous, parent Link2, child Link3, origin xyz=0 -0.0030000000000001 0.0450000000000002 rpy=1.06447174148775 0 0, axis 1 0 0
- added joint Joint2: type continuous, parent Link3, child Link4, origin xyz=0 0 0.204 rpy=-0.982875993996659 0 0, axis -1 0 0
- added joint Joint3: type continuous, parent Link4, child Link5, origin xyz=0 0.00300000000000002 0.0339337982667513 rpy=0 0 -0.0373408822518601, axis 0 0 -1
- added joint Joint4: type continuous, parent Link5, child Link6, origin xyz=0 0.140049941199938 0.0340662017332484 rpy=0 0.0178678459046033 0, axis 0 1 0
- added joint Joint5: type continuous, parent Link6, child Link7, origin xyz=0 0.0509500588000616 0.00300000000000006 rpy=-0.00877434456653207 0 0, axis -1 0 0
- added joint Joint6: type continuous, parent Link7, child EndEffector, origin xyz=0.000999999999997949 0.124829928909805 0 rpy=0 0 0, axis 0 -1 0
